File: Remora Nucleo F446ZE Hat.kicad_pcb (KiCad board)
At the start: 2 copper layers, 80.2 x 133.3 mm, 204 parts, among them J1 NucleoF446ZE CN11 Header, J10 B_STEP_AND_DIR+-, J11 C_STEP_AND_DIR+-, J12 DIGITAL_OUTPUTS, J13 Spindle Out, J14 Digital Inputs, J15 24V Peripheral, J2 NucleoF446ZE CN12 Header, J3 5V_SUPPLY, J3 UART_TX, J4 5V_AUXOUT, J4 MSD-1-A, J5 24V Logic, J6 X_STEP_AND_DIR+-, J7 Y_STEP_AND_DIR+-, J8 Z_STEP_AND_DIR+-, J9 A_STEP_AND_DIR+-, U10 HT26LS31ARZ, U10 LTV-817S, U11 ADuM1201AR, U11 LTV-817S, U12 ADuM1201AR, U12 LTV-817S, U13 HT26LS31ARZ, U13 LTV-817S, U14 ADuM1200AR, U14 ADuM1201AR, U15 ADuM1200AR, U15 ADuM1201AR, U16 ADuM1201AR, U16 HT26LS31ARZ, U17 ADuM1200AR, U17 ADuM1201AR, U18 ADuM1200AR, U18 ADuM1201AR, U19 ADuM1201AR, U19 HT26LS31ARZ, U2 TPS5430DDAR, U20 LTV-817S, U21 LTV-817S, U22 LTV-817S, U23 LTV-817S, U26 ADuM1200AR, U27 ADuM1200AR, U28 ADuM1200AR, U29 ADuM1200AR, U3 TPS5430DDAR, U30 ADuM1200AR, U31 ADuM1200AR, U32 ADuM1200AR, U33 ADuM1200AR, U34 ADuM1200AR, U35 ADuM1200AR, U36 ADuM1200AR, U37 ADuM1200AR, U38 ADuM1200AR, U39 ADuM1200AR, U4 TPS5430DDAR, U40 LTV-817S, U42 TL431DBZ, U5 ADuM1200AR, U5 ADuM1201AR, U6 ADuM1200AR, U6 ADuM1201AR, U7 ADuM1201AR, U7 HT26LS31ARZ, U8 ADuM1201AR, U8 LTV-817S, U9 LTV-817S

Commit message: updates to read me, marked V1 parts inactive and made start on board layout for initial test board. fixes to BOM to suit
Parts:
- removed C1, C3: 10uF, Capacitor_SMD:C_1206_3216Metric_Pad1.33x1.80mm_HandSolder
- removed C10 (x2), C11 (x2), C12 (x2), C13 (x2), C14 (x2), C15 (x2), C16 (x2), C17 (x2), C18 (x2), C19 (x2), C20 (x2), C21 (x2), C23, C25 (x2), C26 (x2), C27 (x2), C28 (x2), C29 (x2), C30 (x2), C31 (x2), C32 (x2), C33 (x2), C34, C35, C36, C37, C38, C39, C40, C41, C42, C43, C44, C45, C46, C47, C48, C49, C50, C51, C52: 100nF, Capacitor_SMD:C_1206_3216Metric_Pad1.33x1.80mm_HandSolder
- removed C2, C5, C8: 10nF, Capacitor_SMD:C_1206_3216Metric_Pad1.33x1.80mm_HandSolder
- removed the C22 at (-109.2, 58.7)
- removed the C22 at (-166.9, 157.7)
- removed the C24 at (-187.8, 157.7)
- removed C6: 4.7uF, Capacitor_SMD:C_1206_3216Metric_Pad1.33x1.80mm_HandSolder
- removed D2, D3, D4: B340A, Diode_SMD:D_1206_3216Metric_Pad1.42x1.75mm_HandSolder
- removed D4: RXLED, Diode_SMD:D_1206_3216Metric_Pad1.42x1.75mm_HandSolder
- removed D5: 12VLED, Diode_SMD:D_1206_3216Metric_Pad1.42x1.75mm_HandSolder
- removed D6: 5VLED, Diode_SMD:D_1206_3216Metric_Pad1.42x1.75mm_HandSolder
- removed D7: 3V3LED, Diode_SMD:D_1206_3216Metric_Pad1.42x1.75mm_HandSolder
- removed F1, F10, F2, F3, F4, F5, F6, F7, F8, F9: 45mA Resettable Fuse (PRG18BB101MB1RB), Fuse:Fuse_0603_1608Metric_Pad1.05x0.95mm_HandSolder
- removed J13: Spindle Out, EBWA_02_A:ADAMTECH_EBWA-02-A
- removed J15: 24V Peripheral, EBWA_02_A:ADAMTECH_EBWA-02-A
- removed the J3 at (176.5, 82.5)
- removed the J4 at (171.2, 37.4)
- removed J5: 24V Logic, EBWA_02_A:ADAMTECH_EBWA-02-A
- removed JP1 (x2): EXT_5V_SUPPLY_JMP, Jumper:SolderJumper-2_P1.3mm_Open_TrianglePad1.0x1.5mm
- removed JP2 (x2): EXT_5V_GND_JMP, Jumper:SolderJumper-2_P1.3mm_Open_TrianglePad1.0x1.5mm
- removed R10, R7: 100R, Resistor_SMD:R_1206_3216Metric_Pad1.30x1.75mm_HandSolder
- removed R11, R12, R13, R14, R15, R16, R20, R21, R22, R23, R27: 82R, Resistor_SMD:R_1206_3216Metric_Pad1.30x1.75mm_HandSolder
- removed R2, R4, R8: 10K 1%, Resistor_SMD:R_1206_3216Metric_Pad1.30x1.75mm_HandSolder
- removed R24, R28: 10K, Resistor_SMD:R_1206_3216Metric_Pad1.30x1.75mm_HandSolder
- removed R29: 30K, Resistor_SMD:R_1206_3216Metric_Pad1.30x1.75mm_HandSolder
- removed R3: 3K2 1%, Resistor_SMD:R_1206_3216Metric_Pad1.30x1.75mm_HandSolder
- removed R5: 1K 1%, Resistor_SMD:R_1206_3216Metric_Pad1.30x1.75mm_HandSolder
- removed R6: 500R, Resistor_SMD:R_1206_3216Metric_Pad1.30x1.75mm_HandSolder
- removed R7: 150R, Resistor_SMD:R_1206_3216Metric_Pad1.30x1.75mm_HandSolder
- removed R9: 5K6 1%, Resistor_SMD:R_1206_3216Metric_Pad1.30x1.75mm_HandSolder
- removed RV1, RV2: 50R trimpot, Potentiometer_SMD:Potentiometer_Bourns_3224W_Vertical
- removed RV3: 500R trimpot, Potentiometer_SMD:Potentiometer_Bourns_3224W_Vertical
- removed U10, U13: HT26LS31ARZ, Package_SO:SOIC-16_3.9x9.9mm_P1.27mm
- removed U10, U11, U12, U13, U20, U21, U22, U23, U40, U8, U9: LTV-817S, Package_SO:SOIC-16_3.9x9.9mm_P1.27mm
- removed U11, U12, U14, U15, U16, U17, U18, U19, U5, U6, U7, U8: ADuM1201AR, Package_SO:SOIC-8_3.9x4.9mm_P1.27mm
- removed U14, U15, U17, U18, U26, U27, U28, U29, U30, U31, U32, U33, U34, U35, U36, U37, U38, U39, U5, U6: ADuM1200AR, Package_SO:SOIC-8_3.9x4.9mm_P1.27mm
- removed U16, U19, U7: HT26LS31ARZ, Package_DIP:SMDIP-4_W9.53mm
- removed U2, U3, U4: TPS5430DDAR, Package_SO:TI_SO-PowerPAD-8_ThermalVias
- removed U42: TL431DBZ, Package_TO_SOT_SMD:SOT-23
- added C22: 100nF, Capacitor_SMD:C_1206_3216Metric_Pad1.33x1.80mm_HandSolder, F.Cu at (195.6, 77.5)
- added SW2: SW_Push, Button_Switch_SMD:SW_SPST_Omron_B3FS-100xP, F.Cu at (98.8, 41.1)
- J3: value 5V_SUPPLY -> UART_TX; footprint OSTVTerminalBlocks:Conn01x02 -> Connector_PinHeader_2.54mm:PinHeader_1x02_P2.54mm_Vertical
- J4: value 5V_AUXOUT -> MSD-1-A; footprint OSTVTerminalBlocks:Conn01x02 -> MSD1A Symbols:MSD1A
- moved J9 396.3 mm to (194.3, 125.7), turned to 90 degrees
- moved J8 388.6 mm to (181.6, 125.7), turned to 90 degrees
- moved J11 360.4 mm to (194.3, 100.3), turned to 90 degrees
- moved J7 358.6 mm to (194.3, 150.5), turned to 90 degrees
- moved J6 351.8 mm to (181.6, 150.5), turned to 90 degrees
- moved J10 351.5 mm to (181.6, 100.3), turned to 90 degrees
- moved J12 306.2 mm to (195.6, 73.7), turned to 90 degrees
- moved J3 287.7 mm to (179.1, 72.4), turned to 90 degrees
- moved J4 275.8 mm to (172.7, 36.9), turned to 180 degrees
- moved C24 259.2 mm to (105.4, 45.7), turned to 90 degrees
- moved J14 232.7 mm to (98.3, 50.4), turned to -90 degrees
- moved R19 200.9 mm to (98.8, 33.0), turned to 180 degrees
- moved R17 141.8 mm to (173.0, 156.8), turned to 180 degrees
- moved D8 140.4 mm to (167.3, 156.8), turned to 0 degrees
- moved C54 32.7 mm to (163.6, 48.3), turned to -90 degrees
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Connections:
- net MCU_RST renamed /MCU_RST
- C24 pad 2: GNDPWR -> GNDREF
- J1 pad 11: unconnected-(J1-Pin_11-Pad11) -> MCU_DIGITAL_IN_2
- J1 pad 17: unconnected-(J1-Pin_17-Pad17) -> MCU_DIGITAL_IN_3
- J1 pad 21: unconnected-(J1-Pin_21-Pad21) -> MCU_DIGITAL_IN_4
- J1 pad 23: USR_BTN -> MCU_DIGITAL_IN_5
- J1 pad 25: unconnected-(J1-Pin_25-Pad25) -> MCU_DIGITAL_IN_6
- J1 pad 27: unconnected-(J1-Pin_27-Pad27) -> MCU_DIGITAL_IN_7
- J1 pad 28: unconnected-(J1-Pin_28-Pad28) -> MCU_DIGITAL_IN_8
- J1 pad 29: unconnected-(J1-Pin_29-Pad29) -> MCU_DIGITAL_IN_9
- J1 pad 30: unconnected-(J1-Pin_30-Pad30) -> MCU_DIGITAL_IN_10
- J1 pad 31: unconnected-(J1-Pin_31-Pad31) -> MCU_DIGITAL_IN_11
- J1 pad 34: unconnected-(J1-Pin_34-Pad34) -> MCU_DIGITAL_IN_12
- J1 pad 35: unconnected-(J1-Pin_35-Pad35) -> MCU_DIGITAL_IN_13
- J1 pad 36: unconnected-(J1-Pin_36-Pad36) -> MCU_DIGITAL_IN_14
- J1 pad 37: unconnected-(J1-Pin_37-Pad37) -> MCU_DIGITAL_IN_15
- J1 pad 38: unconnected-(J1-Pin_38-Pad38) -> MCU_DIGITAL_IN_16
- J1 pad 39: unconnected-(J1-Pin_39-Pad39) -> MCU_DIGITAL_IN_17
- J1 pad 40: unconnected-(J1-Pin_40-Pad40) -> MCU_DIGITAL_IN_18
- J1 pad 41: unconnected-(J1-Pin_41-Pad41) -> MCU_DIGITAL_IN_19
- J1 pad 42: unconnected-(J1-Pin_42-Pad42) -> MCU_DIGITAL_IN_20
- J1 pad 43: unconnected-(J1-Pin_43-Pad43) -> MCU_DIGITAL_IN_21
- J1 pad 44: unconnected-(J1-Pin_44-Pad44) -> MCU_DIGITAL_IN_22
- J1 pad 45: unconnected-(J1-Pin_45-Pad45) -> MCU_DIGITAL_IN_23
- J1 pad 46: unconnected-(J1-Pin_46-Pad46) -> MCU_DIGITAL_IN_24
- J1 pad 47: unconnected-(J1-Pin_47-Pad47) -> MCU_DIGITAL_IN_25
- J1 pad 48: unconnected-(J1-Pin_48-Pad48) -> MCU_DIGITAL_IN_26
- J1 pad 50: unconnected-(J1-Pin_50-Pad50) -> MCU_DIGITAL_IN_28
- J1 pad 51: unconnected-(J1-Pin_51-Pad51) -> MCU_DIGITAL_IN_27
- J1 pad 9: unconnected-(J1-Pin_9-Pad9) -> MCU_DIGITAL_IN_1
- J10 pad 2: /B and C Stepper Drivers/B_STEP+ -> /MCU_B_STEP
- J10 pad 3: /B and C Stepper Drivers/B_STEP- -> unconnected-(J10-Pin_3-Pad3)
- J10 pad 4: /B and C Stepper Drivers/B_DIR+ -> /MCU_B_DIR
- J10 pad 5: /B and C Stepper Drivers/B_DIR- -> unconnected-(J10-Pin_5-Pad5)
- J10 pad 6: GNDPWR -> GNDREF
- J11 pad 2: /B and C Stepper Drivers/C_STEP+ -> /MCU_C_STEP
- J11 pad 3: /B and C Stepper Drivers/C_STEP- -> unconnected-(J11-Pin_3-Pad3)
- J11 pad 4: /B and C Stepper Drivers/C_DIR+ -> /MCU_C_DIR
- J11 pad 5: /B and C Stepper Drivers/C_DIR- -> unconnected-(J11-Pin_5-Pad5)
- J11 pad 6: GNDPWR -> GNDREF
- J12 pad 10: /Digital Outputs/1CH digital output driver 9/OUTPUT9 -> MCU_DIGITAL_OUT_9
- J12 pad 11: /Digital Outputs/1CH digital output driver 10/OUTPUT10 -> MCU_DIGITAL_OUT_10
- J12 pad 12: GNDPWR -> GNDREF
- J12 pad 2: /Digital Outputs/1CH digital output driver 1/OUTPUT1 -> MCU_DIGITAL_OUT_1
- J12 pad 3: /Digital Outputs/1CH digital output driver 2/OUTPUT2 -> MCU_DIGITAL_OUT_2
- J12 pad 4: /Digital Outputs/1CH digital output driver 3/OUTPUT3 -> MCU_DIGITAL_OUT_3
- J12 pad 5: /Digital Outputs/1CH digital output driver 4/OUTPUT4 -> MCU_DIGITAL_OUT_4
- J12 pad 6: /Digital Outputs/1CH digital output driver 5/OUTPUT5 -> MCU_DIGITAL_OUT_5
- J12 pad 7: /Digital Outputs/1CH digital output driver 6/OUTPUT6 -> MCU_DIGITAL_OUT_6
- J12 pad 8: /Digital Outputs/1CH digital output driver 7/OUTPUT7 -> MCU_DIGITAL_OUT_7
- J12 pad 9: /Digital Outputs/1CH digital output driver 8/OUTPUT8 -> MCU_DIGITAL_OUT_8
- J14 pad 10: /Inputs/Digital Input 9&10/MCU_IP9 -> MCU_DIGITAL_IN_9
- J14 pad 11: /Inputs/Digital Input 9&10/MCU_IP10 -> MCU_DIGITAL_IN_10
- J14 pad 12: /Inputs/Digital Input 11&12/MCU_IP11 -> MCU_DIGITAL_IN_11
- J14 pad 13: /Inputs/Digital Input 11&12/MCU_IP12 -> MCU_DIGITAL_IN_12
- J14 pad 14: unconnected-(J14-Pin_14-Pad14) -> MCU_DIGITAL_IN_13
- J14 pad 15: unconnected-(J14-Pin_15-Pad15) -> MCU_DIGITAL_IN_14
- J14 pad 16: /Inputs/Digital Input 15&16/MCU_IP15 -> MCU_DIGITAL_IN_15
- J14 pad 17: /Inputs/Digital Input 15&16/MCU_IP16 -> MCU_DIGITAL_IN_16
- J14 pad 18: /Inputs/Digital Input 17&18/MCU_IP17 -> MCU_DIGITAL_IN_17
- J14 pad 19: /Inputs/Digital Input 17&18/MCU_IP18 -> MCU_DIGITAL_IN_18
- J14 pad 2: /Inputs/Digital Input 1&2/MCU_IP1 -> MCU_DIGITAL_IN_1
- J14 pad 20: /Inputs/Digital Input 19&20/MCU_IP19 -> MCU_DIGITAL_IN_19
- J14 pad 21: /Inputs/Digital Input 19&20/MCU_IP20 -> MCU_DIGITAL_IN_20
- J14 pad 22: unconnected-(J14-Pin_22-Pad22) -> MCU_DIGITAL_IN_21
- J14 pad 23: unconnected-(J14-Pin_23-Pad23) -> MCU_DIGITAL_IN_22
- J14 pad 24: /Inputs/Digital Input 23&24/MCU_IP23 -> MCU_DIGITAL_IN_23
- J14 pad 25: /Inputs/Digital Input 23&24/MCU_IP24 -> MCU_DIGITAL_IN_24
- J14 pad 26: /Inputs/Digital Input 25&26/MCU_IP25 -> MCU_DIGITAL_IN_25
- J14 pad 27: /Inputs/Digital Input 25&26/MCU_IP26 -> MCU_DIGITAL_IN_26
- J14 pad 28: /Inputs/Digital Input 27&28/MCU_IP27 -> MCU_DIGITAL_IN_27
- J14 pad 29: /Inputs/Digital Input 27&28/MCU_IP28 -> MCU_DIGITAL_IN_28
- J14 pad 3: /Inputs/Digital Input 1&2/MCU_IP2 -> MCU_DIGITAL_IN_2
- J14 pad 30: GNDPWR -> GNDREF
- J14 pad 4: /Inputs/Digital Input 3&4/MCU_IP3 -> MCU_DIGITAL_IN_3
- J14 pad 5: /Inputs/Digital Input 3&4/MCU_IP4 -> MCU_DIGITAL_IN_4
- J14 pad 6: /Inputs/Digital Input 5&6/MCU_IP5 -> MCU_DIGITAL_IN_5
- J14 pad 7: /Inputs/Digital Input 5&6/MCU_IP6 -> MCU_DIGITAL_IN_6
- J14 pad 8: /Inputs/Digital Input 7&8/MCU_IP7 -> MCU_DIGITAL_IN_7
- J14 pad 9: /Inputs/Digital Input 7&8/MCU_IP8 -> MCU_DIGITAL_IN_8
- J2 pad 12: unconnected-(J2-Pin_12-Pad12) -> MCU_DIGITAL_OUT_8
- J2 pad 14: unconnected-(J2-Pin_14-Pad14) -> MCU_DIGITAL_OUT_7
- J2 pad 16: unconnected-(J2-Pin_16-Pad16) -> MCU_DIGITAL_OUT_6
- J2 pad 18: unconnected-(J2-Pin_18-Pad18) -> MCU_DIGITAL_OUT_5
- J2 pad 22: unconnected-(J2-Pin_22-Pad22) -> MCU_DIGITAL_OUT_4
- J2 pad 24: unconnected-(J2-Pin_24-Pad24) -> MCU_DIGITAL_OUT_3
- J2 pad 26: unconnected-(J2-Pin_26-Pad26) -> MCU_DIGITAL_OUT_2
- J2 pad 28: USR_LED -> MCU_DIGITAL_OUT_1
- J2 pad 4: unconnected-(J2-Pin_4-Pad4) -> MCU_DIGITAL_OUT_10
- J2 pad 55: unconnected-(J2-Pin_55-Pad55) -> /MCU_B_DIR
- J2 pad 57: unconnected-(J2-Pin_57-Pad57) -> /MCU_B_STEP
- J2 pad 59: unconnected-(J2-Pin_59-Pad59) -> /MCU_Z_DIR
- J2 pad 6: unconnected-(J2-Pin_6-Pad6) -> MCU_DIGITAL_OUT_9
- J2 pad 60: unconnected-(J2-Pin_60-Pad60) -> /MCU_C_DIR
- J2 pad 61: unconnected-(J2-Pin_61-Pad61) -> /MCU_Z_STEP
- J2 pad 62: unconnected-(J2-Pin_62-Pad62) -> /MCU_C_STEP
- J2 pad 64: unconnected-(J2-Pin_64-Pad64) -> /MCU_A_DIR
- J2 pad 65: unconnected-(J2-Pin_65-Pad65) -> /USR_LED
- J2 pad 66: unconnected-(J2-Pin_66-Pad66) -> /MCU_A_STEP
- J2 pad 67: unconnected-(J2-Pin_67-Pad67) -> /MCU_X_DIR
- J2 pad 68: unconnected-(J2-Pin_68-Pad68) -> /MCU_Y_DIR
- J2 pad 69: unconnected-(J2-Pin_69-Pad69) -> /MCU_X_STEP
- J2 pad 70: unconnected-(J2-Pin_70-Pad70) -> /MCU_Y_STEP
- J3 pad 1: +5VD -> GNDREF
- J3 pad 2: 5V_GND -> /UART_TX
- J4 pad 1: +5VD -> /SDIO_D2
- J4 pad 2: 5V_GND -> /SDIO_D3
- J6 pad 2: /X and Y Stepper Drivers/X_STEP+ -> /MCU_X_STEP
- J6 pad 3: /X and Y Stepper Drivers/X_STEP- -> unconnected-(J6-Pin_3-Pad3)
- J6 pad 4: /X and Y Stepper Drivers/X_DIR+ -> /MCU_X_DIR
- J6 pad 5: /X and Y Stepper Drivers/X_DIR- -> unconnected-(J6-Pin_5-Pad5)
- J6 pad 6: GNDPWR -> GNDREF
- J7 pad 2: /X and Y Stepper Drivers/Y_STEP+ -> /MCU_Y_STEP
- J7 pad 3: /X and Y Stepper Drivers/Y_STEP- -> unconnected-(J7-Pin_3-Pad3)
- J7 pad 4: /X and Y Stepper Drivers/Y_DIR+ -> /MCU_Y_DIR
- J7 pad 5: /X and Y Stepper Drivers/Y_DIR- -> unconnected-(J7-Pin_5-Pad5)
- J7 pad 6: GNDPWR -> GNDREF
- J8 pad 2: /Z and A Stepper Drivers/Z_STEP+ -> /MCU_Z_STEP
- J8 pad 3: /Z and A Stepper Drivers/Z_STEP- -> unconnected-(J8-Pin_3-Pad3)
- J8 pad 4: /Z and A Stepper Drivers/Z_DIR+ -> /MCU_Z_DIR
- J8 pad 5: /Z and A Stepper Drivers/Z_DIR- -> unconnected-(J8-Pin_5-Pad5)
- J8 pad 6: GNDPWR -> GNDREF
- J9 pad 2: /Z and A Stepper Drivers/A_STEP+ -> /MCU_A_STEP
- J9 pad 3: /Z and A Stepper Drivers/A_STEP- -> unconnected-(J9-Pin_3-Pad3)
- J9 pad 4: /Z and A Stepper Drivers/A_DIR+ -> /MCU_A_DIR
- J9 pad 5: /Z and A Stepper Drivers/A_DIR- -> unconnected-(J9-Pin_5-Pad5)
- J9 pad 6: GNDPWR -> GNDREF
- R17 pad 1: USR_LED -> /USR_LED
- U1 pad 2: /WIZ_CS -> /SPI1_CS
Routing:
- net +5VD: track 0.00 -> 177.5 mm
- net /SDIO_CLK: track 0.00 -> 80.5 mm, vias 0 -> 1
- net /SDIO_CMD: track 0.00 -> 76.6 mm, vias 0 -> 1
- net /SDIO_D2: track 0.00 -> 73.6 mm, vias 0 -> 1
- net /SDIO_D3: track 0.00 -> 72.5 mm, vias 0 -> 1
- net /MCU_C_DIR: track 0.00 -> 67.4 mm
- net /MCU_C_STEP: track 0.00 -> 65.8 mm
- net /MCU_B_STEP: track 0.00 -> 57.2 mm
- net /MCU_RST: track 0.00 -> 55.9 mm
- net /MCU_B_DIR: track 0.00 -> 53.0 mm
- net MCU_DIGITAL_OUT_7: track 0.00 -> 45.1 mm
- net MCU_DIGITAL_OUT_6: track 0.00 -> 43.9 mm
- net MCU_DIGITAL_OUT_8: track 0.00 -> 43.6 mm
- net MCU_DIGITAL_OUT_5: track 0.00 -> 42.7 mm
- net +3V3: track 0.00 -> 42.7 mm
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- added copper zone on B.Cu, net GNDREF
- added copper zone on F.Cu, net GNDREF
Other:
- board size 80.2 x 133.3 mm -> 108.2 x 137.1 mm
- board text added: "1"
- board text added: "10"
- board text added: "11"
- board text added: "12"
- board text added: "13"
- board text added: "14"
- board text added: "15"
- board text added: "16"
- board text added: "17"
- board text added: "18"
- board text added: "19"
- board text added: "2"
- board text added: "20"
- board text added: "21"
- board text added: "22"
- board text added: "23"
- board text added: "24"
- board text added: "25"
- board text added: "26"
- board text added: "27"
- board text added: "28"
- board text added: "3"
- board text added: "4"
- board text added: "5"
- board text added: "5V"
- board text added: "6"
- board text added: "7"
- board text added: "8"
- board text added: "9"
- board text added: "A_Step"
- board text added: "B_Step"
- board text added: "C_Step"
- board text added: "DIR+"
- board text added: "DIR-"
- board text added: "GND"
- board text added: "ST+"
- board text added: "ST-"
- board text added: "UART TX"
- board text added: "USR LED"
- board text added: "X_Step"
- board text added: "Y_Step"
- board text added: "Z_Step"
