File: Remora Nucleo F446ZE Hat.kicad_pcb (KiCad board)
At the start: 2 copper layers, 138 x 162 mm, 203 parts, among them J1 Conn_02x35_Odd_Even, J10 Conn_01x02_Socket, J11 Conn_01x04_Socket, J12 Conn_01x02_Socket, J13 Conn_01x04_Socket, J14 Conn_01x02_Socket, J15 Conn_01x04_Socket, J16 Conn_01x02_Socket, J17 Conn_01x04_Socket, J18 Conn_01x02_Socket, J19 Conn_01x04_Socket, J20 Conn_01x04_Socket, J21 Conn_01x02_Socket, J22 Conn_01x04_Socket, J23 Conn_01x04_Socket, J24 Conn_01x02_Socket, J25 Spindle Out, J26 Conn_01x04_Socket, J27 Conn_01x04_Socket, J28 Conn_01x04_Socket, J29 Conn_01x04_Socket, J3 UART_TX, J30 Conn_01x02_Socket, J4 Conn_02x35_Odd_Even, J5 24V Logic, J6 24V Isolated, J7 Conn_01x04_Socket, J8 Conn_01x02_Socket, J9 Conn_01x04_Socket, Q1 BC847, SW1 SW_Push, U1 Wiznet W5500 Eval Module, U10 LTV-247, U11 LTV-247, U12 LTV-247, U13 AM26LS31CDR, U14 LTV-247, U15 AM26LS31CDR, U16 MCP6042, U17 LTV-247, U18 TL431A, U2 XL1509-12, U3 XL1509-5.0, U4 LTV-247, U5 AM26LS31CDR, U6 LTV-247, U7 LTV-247, U8 LTV-247, U9 LTV-247

Commit message: Redo of layout to use smaller terminals, applied to steppers and inputs and laid out outputs too
Parts:
- moved C12 378.6 mm to (249.5, 203.6)
- moved C21 357.4 mm to (249.5, 127.6)
- moved J8 356.7 mm to (259.4, 192.8)
- moved J7 353.9 mm to (248.9, 192.8)
- moved C14 344.4 mm to (275.5, 203.5)
- moved R21 344.4 mm to (283.5, 203.6)
- moved R23 344.4 mm to (279.5, 203.6)
- moved R25 344.4 mm to (271.5, 203.6)
- moved R27 344.4 mm to (267.5, 203.6)
- moved J10 343.1 mm to (285.4, 192.8)
- moved C9 341.3 mm to (258.0, 210.0)
- moved R16 341.3 mm to (263.4, 211.8)
- moved R17 341.3 mm to (263.4, 215.1)
- moved R18 341.3 mm to (263.4, 218.4)
- moved R19 341.3 mm to (263.4, 221.7)
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Routing:
- net GNDREF: vias 20 -> 19
Other:
- board text added: "JLCJLCJLCJLC"
- board text added: "© 2026 Ben Jacobson"
- board text removed: "© 2026 Ben Jacobson JLCJLCJLCJLC"
