File: DigitalOutputs.kicad_sch (KiCad schematic)
At the start: 4 parts, among them J22 Conn_01x04_Socket, J23 Conn_01x04_Socket, J24 Conn_01x02_Socket

Commit message: Layout for stepper drivers and digital inputs
Parts:
- renumbered C30 to C33
Changed lines of the file:
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@@
 		(on_board yes)
 		(dnp no)
-		(property "Reference" "C30"
+		(property "Reference" "C33"
 			(at 216.408 74.422 0)
 			(effects
@@
 			(project "Remora Nucleo F446ZE Hat"
 				(path "/5473abc6-7b93-43cc-a401-f691c4d7d7cf/a10f9653-3098-46b3-8571-958500eea49a"
-					(reference "C30")
+					(reference "C33")
 					(unit 1)
 				)
@@
 		(on_board yes)
 		(dnp no)
-		(property "Reference" "#PWR0206"
+		(property "Reference" "#PWR0209"
 			(at 212.09 86.36 0)
 			(effects
@@
 			(project "Remora Nucleo F446ZE Hat"
 				(path "/5473abc6-7b93-43cc-a401-f691c4d7d7cf/a10f9653-3098-46b3-8571-958500eea49a"
-					(reference "#PWR0206")
+					(reference "#PWR0209")
 					(unit 1)
 				)
@@
 		(dnp no)
 		(fields_autoplaced yes)
-		(property "Reference" "#PWR0204"
+		(property "Reference" "#PWR0207"
 			(at 199.39 114.3 0)
 			(effects
@@
 			(project ""
 				(path "/5473abc6-7b93-43cc-a401-f691c4d7d7cf/a10f9653-3098-46b3-8571-958500eea49a"
-					(reference "#PWR0204")
+					(reference "#PWR0207")
 					(unit 1)
 				)
@@
 		(on_board yes)
 		(dnp no)
-		(property "Reference" "#PWR0205"
+		(property "Reference" "#PWR0208"
 			(at 212.09 73.66 0)
 			(effects
@@
 			(project "Remora Nucleo F446ZE Hat"
 				(path "/5473abc6-7b93-43cc-a401-f691c4d7d7cf/a10f9653-3098-46b3-8571-958500eea49a"
-					(reference "#PWR0205")
-					(unit 1)
-				)
+					(reference "#PWR0208")
+					(unit 1)
+				)

Commit message: Switched terminal footprints over to a finer pitch. Corrected an issue with component reference values preventing proper use of multi channel rule areas. Component references for 4 channel optos are more straightforward as a result
Parts:
- J14: renamed from J22; footprint Amphenol QT:QT04ADP83V0000G -> 691412120004B:691412120004B; Digikey Part Number 1818-QT04ADP83V0000G-ND -> 732-691412120004B-ND; Digikey URL https://www.digikey.com.au/en/products/detail/amphenol-anyt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 -> https://www.digikey.com.au/en/products/detail/w%C3%BCrth-el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
- J15: renamed from J23; footprint Amphenol QT:QT04ADP83V0000G -> 691412120004B:691412120004B; Digikey Part Number 1818-QT04ADP83V0000G-ND -> 732-691412120004B-ND; Digikey URL https://www.digikey.com.au/en/products/detail/amphenol-anyt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 -> https://www.digikey.com.au/en/products/detail/w%C3%BCrth-el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
- J16: renamed from J24; footprint Amphenol QT:QT02ADP83V0000G -> 691412120002B:691412120002B; Digikey Part Number 1818-QT02ADP83V0000G-ND -> 732-691412120002B-ND; Digikey URL https://www.digikey.com.au/en/products/detail/amphenol-anyt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 -> https://www.digikey.com.au/en/products/detail/w%C3%BCrth-el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
- renumbered C33 to C21
Changed lines of the file:
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@@
 		(on_board yes)
 		(dnp no)
-		(property "Reference" "C33"
+		(property "Reference" "C21"
 			(at 216.408 74.422 0)
 			(effects
@@
 			(project "Remora Nucleo F446ZE Hat"
 				(path "/5473abc6-7b93-43cc-a401-f691c4d7d7cf/a10f9653-3098-46b3-8571-958500eea49a"
-					(reference "C33")
+					(reference "C21")
 					(unit 1)
 				)
@@
 		(on_board yes)
 		(dnp no)
-		(property "Reference" "#PWR0209"
+		(property "Reference" "#PWR0149"
 			(at 212.09 86.36 0)
 			(effects
@@
 			(project "Remora Nucleo F446ZE Hat"
 				(path "/5473abc6-7b93-43cc-a401-f691c4d7d7cf/a10f9653-3098-46b3-8571-958500eea49a"
-					(reference "#PWR0209")
+					(reference "#PWR0149")
 					(unit 1)
 				)
@@
 		(on_board yes)
 		(dnp no)
-		(property "Reference" "J23"
+		(property "Reference" "J15"
 			(at 219.964 94.742 0)
 			(effects
@@
 			)
 		)
-		(property "Footprint" "Amphenol QT:QT04ADP83V0000G"
+		(property "Footprint" "691412120004B:691412120004B"
 			(at 205.74 96.52 0)
 			(effects
@@
 			)
 		)
-		(property "Digikey Part Number" "1818-QT04ADP83V0000G-ND"
+		(property "Digikey Part Number" "732-691412120004B-ND"
 			(at 205.74 96.52 0)
 			(effects
@@
 			)
 		)
-		(property "Digikey URL" "https://www.digikey.com.au/en/products/detail/amphenol-anytek/QT04ADP83V0000G/25618782"
+		(property "Digikey URL" "https://www.digikey.com.au/en/products/detail/w%C3%BCrth-elektronik/691412120004B/11478393"
 			(at 205.74 96.52 0)
 			(effects
@@
 			(project "Remora Nucleo F446ZE Hat"
 				(path "/5473abc6-7b93-43cc-a401-f691c4d7d7cf/a10f9653-3098-46b3-8571-958500eea49a"
-					(reference "J23")
+					(reference "J15")
 					(unit 1)
 				)
@@
 		(on_board yes)
 		(dnp no)
-		(property "Reference" "J22"
+		(property "Reference" "J14"
 			(at 219.964 88.392 0)
 			(effects
@@
 			)
 		)
-		(property "Footprint" "Amphenol QT:QT04ADP83V0000G"
+		(property "Footprint" "691412120004B:691412120004B"
 			(at 205.74 86.36 0)
 			(effects
@@
 			)
 		)
-		(property "Digikey Part Number" "1818-QT04ADP83V0000G-ND"
+		(property "Digikey Part Number" "732-691412120004B-ND"
 			(at 205.74 86.36 0)
 			(effects
@@
 			)
 		)
-		(property "Digikey URL" "https://www.digikey.com.au/en/products/detail/amphenol-anytek/QT04ADP83V0000G/25618782"
+		(property "Digikey URL" "https://www.digikey.com.au/en/products/detail/w%C3%BCrth-elektronik/691412120004B/11478393"
 			(at 205.74 86.36 0)
 			(effects
@@
 			(project "Remora Nucleo F446ZE Hat"
 				(path "/5473abc6-7b93-43cc-a401-f691c4d7d7cf/a10f9653-3098-46b3-8571-958500eea49a"
-					(reference "J22")
+					(reference "J14")
 					(unit 1)
 				)
@@
 		(dnp no)
 		(fields_autoplaced yes)
-		(property "Reference" "#PWR0207"
+		(property "Reference" "#PWR0147"
 			(at 199.39 114.3 0)
 			(effects
@@
 			(project ""
 				(path "/5473abc6-7b93-43cc-a401-f691c4d7d7cf/a10f9653-3098-46b3-8571-958500eea49a"
-					(reference "#PWR0207")
+					(reference "#PWR0147")
 					(unit 1)
 				)
@@
 		(on_board yes)
 		(dnp no)
-		(property "Reference" "#PWR0208"
+		(property "Reference" "#PWR0148"
 			(at 212.09 73.66 0)
 			(effects
@@
 			(project "Remora Nucleo F446ZE Hat"
 				(path "/5473abc6-7b93-43cc-a401-f691c4d7d7cf/a10f9653-3098-46b3-8571-958500eea49a"
-					(reference "#PWR0208")
+					(reference "#PWR0148")
 					(unit 1)
 				)
@@
 		(on_board yes)
 		(dnp no)
-		(property "Reference" "J24"
+		(property "Reference" "J16"
 			(at 219.964 101.092 0)
 			(effects
@@
 			)
 		)
-		(property "Footprint" "Amphenol QT:QT02ADP83V0000G"
+		(property "Footprint" "691412120002B:691412120002B"
 			(at 205.74 104.14 0)
 			(effects
@@
 			)
 		)
-		(property "Digikey Part Number" "1818-QT02ADP83V0000G-ND"
+		(property "Digikey Part Number" "732-691412120002B-ND"
 			(at 205.74 104.14 0)
 			(effects
@@
 			)
 		)
-		(property "Digikey URL" "https://www.digikey.com.au/en/products/detail/amphenol-anytek/QT02ADP83V0000G/25618889"
+		(property "Digikey URL" "https://www.digikey.com.au/en/products/detail/w%C3%BCrth-elektronik/691412120002B/11478592"
 			(at 205.74 104.14 0)
 			(effects
@@
 			(project "Remora Nucleo F446ZE Hat"
 				(path "/5473abc6-7b93-43cc-a401-f691c4d7d7cf/a10f9653-3098-46b3-8571-958500eea49a"
-					(reference "J24")
-					(unit 1)
-				)
+					(reference "J16")
+					(unit 1)
+				)

Commit message: Added 3d Models for new terminal connectors for easy board verification before committing to build
Parts:
- renumbered C21 to C33, J14 to J22, J15 to J23, J16 to J24
Changed lines of the file:
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@@
 		(on_board yes)
 		(dnp no)
-		(property "Reference" "C21"
+		(property "Reference" "C33"
 			(at 216.408 74.422 0)
 			(effects
@@
 			(project "Remora Nucleo F446ZE Hat"
 				(path "/5473abc6-7b93-43cc-a401-f691c4d7d7cf/a10f9653-3098-46b3-8571-958500eea49a"
-					(reference "C21")
+					(reference "C33")
 					(unit 1)
 				)
@@
 		(on_board yes)
 		(dnp no)
-		(property "Reference" "#PWR0149"
+		(property "Reference" "#PWR0217"
 			(at 212.09 86.36 0)
 			(effects
@@
 			(project "Remora Nucleo F446ZE Hat"
 				(path "/5473abc6-7b93-43cc-a401-f691c4d7d7cf/a10f9653-3098-46b3-8571-958500eea49a"
-					(reference "#PWR0149")
+					(reference "#PWR0217")
 					(unit 1)
 				)
@@
 		(on_board yes)
 		(dnp no)
-		(property "Reference" "J15"
+		(property "Reference" "J23"
 			(at 219.964 94.742 0)
 			(effects
@@
 			(project "Remora Nucleo F446ZE Hat"
 				(path "/5473abc6-7b93-43cc-a401-f691c4d7d7cf/a10f9653-3098-46b3-8571-958500eea49a"
-					(reference "J15")
+					(reference "J23")
 					(unit 1)
 				)
@@
 		(on_board yes)
 		(dnp no)
-		(property "Reference" "J14"
+		(property "Reference" "J22"
 			(at 219.964 88.392 0)
 			(effects
@@
 			(project "Remora Nucleo F446ZE Hat"
 				(path "/5473abc6-7b93-43cc-a401-f691c4d7d7cf/a10f9653-3098-46b3-8571-958500eea49a"
-					(reference "J14")
+					(reference "J22")
 					(unit 1)
 				)
@@
 		(dnp no)
 		(fields_autoplaced yes)
-		(property "Reference" "#PWR0147"
+		(property "Reference" "#PWR0215"
 			(at 199.39 114.3 0)
 			(effects
@@
 			(project ""
 				(path "/5473abc6-7b93-43cc-a401-f691c4d7d7cf/a10f9653-3098-46b3-8571-958500eea49a"
-					(reference "#PWR0147")
+					(reference "#PWR0215")
 					(unit 1)
 				)
@@
 		(on_board yes)
 		(dnp no)
-		(property "Reference" "#PWR0148"
+		(property "Reference" "#PWR0216"
 			(at 212.09 73.66 0)
 			(effects
@@
 			(project "Remora Nucleo F446ZE Hat"
 				(path "/5473abc6-7b93-43cc-a401-f691c4d7d7cf/a10f9653-3098-46b3-8571-958500eea49a"
-					(reference "#PWR0148")
+					(reference "#PWR0216")
 					(unit 1)
 				)
@@
 		(on_board yes)
 		(dnp no)
-		(property "Reference" "J16"
+		(property "Reference" "J24"
 			(at 219.964 101.092 0)
 			(effects
@@
 			(project "Remora Nucleo F446ZE Hat"
 				(path "/5473abc6-7b93-43cc-a401-f691c4d7d7cf/a10f9653-3098-46b3-8571-958500eea49a"
-					(reference "J16")
-					(unit 1)
-				)
+					(reference "J24")
+					(unit 1)
+				)
