File: SpindleDAC.kicad_sch (KiCad schematic)
At the start: 18 parts, among them J17 Spindle Out, Q1 BC847, U13 LTV-247, U14 TL431A

Commit message: Added 3d Models for new terminal connectors for easy board verification before committing to build
Parts:
- renumbered C22 to C34, C23 to C35, C24 to C36, C25 to C37, J17 to J25, R59 to R91, R60 to R92, R61 to R93, R62 to R94, R63 to R95, R64 to R96, R65 to R97, R66 to R98, U13 to U17, U14 to U18
Changed lines of the file:
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@@
 		(on_board yes)
 		(dnp no)
-		(property "Reference" "R62"
+		(property "Reference" "R94"
 			(at 157.48 117.348 90)
 			(effects
@@
 			(project "Remora Nucleo F446ZE Hat"
 				(path "/5473abc6-7b93-43cc-a401-f691c4d7d7cf/5cdad347-c6ad-4791-9d53-e4d1ad999196"
-					(reference "R62")
+					(reference "R94")
 					(unit 1)
 				)
@@
 		(on_board yes)
 		(dnp no)
-		(property "Reference" "R61"
+		(property "Reference" "R93"
 			(at 134.62 117.348 90)
 			(effects
@@
 			(project "Remora Nucleo F446ZE Hat"
 				(path "/5473abc6-7b93-43cc-a401-f691c4d7d7cf/5cdad347-c6ad-4791-9d53-e4d1ad999196"
-					(reference "R61")
+					(reference "R93")
 					(unit 1)
 				)
@@
 		(dnp no)
 		(fields_autoplaced yes)
-		(property "Reference" "U13"
+		(property "Reference" "U17"
 			(at 110.49 102.87 0)
 			(effects
@@
 			(project ""
 				(path "/5473abc6-7b93-43cc-a401-f691c4d7d7cf/5cdad347-c6ad-4791-9d53-e4d1ad999196"
-					(reference "U13")
+					(reference "U17")
 					(unit 1)
 				)
@@
 		(on_board yes)
 		(dnp no)
-		(property "Reference" "R64"
+		(property "Reference" "R96"
 			(at 172.212 72.136 0)
 			(effects
@@
 			(project "Remora Nucleo F446ZE Hat"
 				(path "/5473abc6-7b93-43cc-a401-f691c4d7d7cf/5cdad347-c6ad-4791-9d53-e4d1ad999196"
-					(reference "R64")
+					(reference "R96")
 					(unit 1)
 				)
@@
 		(on_board yes)
 		(dnp no)
-		(property "Reference" "#PWR0155"
+		(property "Reference" "#PWR0223"
 			(at 189.23 143.51 0)
 			(effects
@@
 			(project "Remora Nucleo F446ZE Hat"
 				(path "/5473abc6-7b93-43cc-a401-f691c4d7d7cf/5cdad347-c6ad-4791-9d53-e4d1ad999196"
-					(reference "#PWR0155")
+					(reference "#PWR0223")
 					(unit 1)
 				)
@@
 		(on_board yes)
 		(dnp no)
-		(property "Reference" "R65"
+		(property "Reference" "R97"
 			(at 192.278 132.08 90)
 			(effects
@@
 			(project "Remora Nucleo F446ZE Hat"
 				(path "/5473abc6-7b93-43cc-a401-f691c4d7d7cf/5cdad347-c6ad-4791-9d53-e4d1ad999196"
-					(reference "R65")
+					(reference "R97")
 					(unit 1)
 				)
@@
 		(on_board yes)
 		(dnp no)
-		(property "Reference" "R66"
+		(property "Reference" "R98"
 			(at 204.216 31.496 0)
 			(effects
@@
 			(project "Remora Nucleo F446ZE Hat"
 				(path "/5473abc6-7b93-43cc-a401-f691c4d7d7cf/5cdad347-c6ad-4791-9d53-e4d1ad999196"
-					(reference "R66")
+					(reference "R98")
 					(unit 1)
 				)
@@
 		(on_board yes)
 		(dnp no)
-		(property "Reference" "C23"
+		(property "Reference" "C35"
 			(at 167.386 95.25 0)
 			(effects
@@
 			(project "Remora Nucleo F446ZE Hat"
 				(path "/5473abc6-7b93-43cc-a401-f691c4d7d7cf/5cdad347-c6ad-4791-9d53-e4d1ad999196"
-					(reference "C23")
+					(reference "C35")
 					(unit 1)
 				)
@@
 		(on_board yes)
 		(dnp no)
-		(property "Reference" "R59"
+		(property "Reference" "R91"
 			(at 91.694 104.14 90)
 			(effects
@@
 			(project "Remora Nucleo F446ZE Hat"
 				(path "/5473abc6-7b93-43cc-a401-f691c4d7d7cf/5cdad347-c6ad-4791-9d53-e4d1ad999196"
-					(reference "R59")
+					(reference "R91")
 					(unit 1)
 				)
@@
 		(dnp no)
 		(fields_autoplaced yes)
-		(property "Reference" "J17"
+		(property "Reference" "J25"
 			(at 231.14 123.1899 0)
 			(effects
@@
 			(project ""
 				(path "/5473abc6-7b93-43cc-a401-f691c4d7d7cf/5cdad347-c6ad-4791-9d53-e4d1ad999196"
-					(reference "J17")
+					(reference "J25")
 					(unit 1)
 				)
@@
 		(dnp no)
 		(fields_autoplaced yes)
-		(property "Reference" "#PWR0150"
+		(property "Reference" "#PWR0218"
 			(at 99.06 134.62 0)
 			(effects
@@
 			(project "Remora Nucleo F446ZE Hat"
 				(path "/5473abc6-7b93-43cc-a401-f691c4d7d7cf/5cdad347-c6ad-4791-9d53-e4d1ad999196"
-					(reference "#PWR0150")
+					(reference "#PWR0218")
 					(unit 1)
 				)
@@
 		(on_board yes)
 		(dnp no)
-		(property "Reference" "C24"
+		(property "Reference" "C36"
 			(at 176.53 127.508 0)
 			(effects
@@
 			(project "Remora Nucleo F446ZE Hat"
 				(path "/5473abc6-7b93-43cc-a401-f691c4d7d7cf/5cdad347-c6ad-4791-9d53-e4d1ad999196"
-					(reference "C24")
+					(reference "C36")
 					(unit 1)
 				)
@@
 		(dnp no)
 		(fields_autoplaced yes)
-		(property "Reference" "#PWR0156"
+		(property "Reference" "#PWR0224"
 			(at 207.01 29.21 0)
 			(effects
@@
 			(project "Remora Nucleo F446ZE Hat"
 				(path "/5473abc6-7b93-43cc-a401-f691c4d7d7cf/5cdad347-c6ad-4791-9d53-e4d1ad999196"
-					(reference "#PWR0156")
+					(reference "#PWR0224")
 					(unit 1)
 				)
@@
 		(on_board yes)
 		(dnp no)
-		(property "Reference" "R63"
+		(property "Reference" "R95"
 			(at 178.562 46.736 90)
 			(effects
@@
 			(project "Remora Nucleo F446ZE Hat"
 				(path "/5473abc6-7b93-43cc-a401-f691c4d7d7cf/5cdad347-c6ad-4791-9d53-e4d1ad999196"
-					(reference "R63")
+					(reference "R95")
 					(unit 1)
 				)
@@
 		(dnp no)
 		(fields_autoplaced yes)
-		(property "Reference" "#PWR0153"
+		(property "Reference" "#PWR0221"
 			(at 161.29 105.41 0)
 			(effects
@@
 			(project "Remora Nucleo F446ZE Hat"
 				(path "/5473abc6-7b93-43cc-a401-f691c4d7d7cf/5cdad347-c6ad-4791-9d53-e4d1ad999196"
-					(reference "#PWR0153")
+					(reference "#PWR0221")
 					(unit 1)
 				)
@@
 		(dnp no)
 		(fields_autoplaced yes)
-		(property "Reference" "U14"
+		(property "Reference" "U18"
 			(at 209.55 52.0699 90)
 			(effects
@@
 			(project ""
 				(path "/5473abc6-7b93-43cc-a401-f691c4d7d7cf/5cdad347-c6ad-4791-9d53-e4d1ad999196"
-					(reference "U14")
+					(reference "U18")
 					(unit 1)
 				)
@@
 		(on_board yes)
 		(dnp no)
-		(property "Reference" "R60"
+		(property "Reference" "R92"
 			(at 128.778 128.27 90)
 			(effects
@@
 			(project "Remora Nucleo F446ZE Hat"
 				(path "/5473abc6-7b93-43cc-a401-f691c4d7d7cf/5cdad347-c6ad-4791-9d53-e4d1ad999196"
-					(reference "R60")
+					(reference "R92")
 					(unit 1)
 				)
@@
 		(dnp no)
 		(fields_autoplaced yes)
-		(property "Reference" "#PWR0158"
+		(property "Reference" "#PWR0226"
 			(at 207.01 106.68 0)
 			(effects
@@
 			(project "Remora Nucleo F446ZE Hat"
 				(path "/5473abc6-7b93-43cc-a401-f691c4d7d7cf/5cdad347-c6ad-4791-9d53-e4d1ad999196"
-					(reference "#PWR0158")
+					(reference "#PWR0226")
 					(unit 1)
 				)
@@
 		(on_board yes)
 		(dnp no)
-		(property "Reference" "#PWR0151"
+		(property "Reference" "#PWR0219"
 			(at 125.73 143.51 0)
 			(effects
@@
 			(project "Remora Nucleo F446ZE Hat"
 				(path "/5473abc6-7b93-43cc-a401-f691c4d7d7cf/5cdad347-c6ad-4791-9d53-e4d1ad999196"
-					(reference "#PWR0151")
+					(reference "#PWR0219")
 					(unit 1)
 				)
@@
 		(dnp no)
 		(fields_autoplaced yes)
-		(property "Reference" "#PWR0159"
+		(property "Reference" "#PWR0227"
 			(at 220.98 143.51 0)
 			(effects
@@
 			(project "Remora Nucleo F446ZE Hat"
 				(path "/5473abc6-7b93-43cc-a401-f691c4d7d7cf/5cdad347-c6ad-4791-9d53-e4d1ad999196"
-					(reference "#PWR0159")
+					(reference "#PWR0227")
 					(unit 1)
 				)
@@
 		(on_board yes)
 		(dnp no)
-		(property "Reference" "C25"
+		(property "Reference" "C37"
 			(at 213.106 96.52 0)
 			(effects
@@
 			(project "Remora Nucleo F446ZE Hat"
 				(path "/5473abc6-7b93-43cc-a401-f691c4d7d7cf/5cdad347-c6ad-4791-9d53-e4d1ad999196"
-					(reference "C25")
+					(reference "C37")
 					(unit 1)
 				)
@@
 		(dnp no)
 		(fields_autoplaced yes)
-		(property "Reference" "#PWR0157"
+		(property "Reference" "#PWR0225"
 			(at 207.01 85.09 0)
 			(effects
@@
 			(project "Remora Nucleo F446ZE Hat"
 				(path "/5473abc6-7b93-43cc-a401-f691c4d7d7cf/5cdad347-c6ad-4791-9d53-e4d1ad999196"
-					(reference "#PWR0157")
+					(reference "#PWR0225")
 					(unit 1)
 				)
@@
 		(dnp no)
 		(fields_autoplaced yes)
-		(property "Reference" "#PWR0152"
+		(property "Reference" "#PWR0220"
 			(at 146.05 143.51 0)
 			(effects
@@
 			(project "Remora Nucleo F446ZE Hat"
 				(path "/5473abc6-7b93-43cc-a401-f691c4d7d7cf/5cdad347-c6ad-4791-9d53-e4d1ad999196"
-					(reference "#PWR0152")
+					(reference "#PWR0220")
 					(unit 1)
 				)
@@
 		(on_board yes)
 		(dnp no)
-		(property "Reference" "C22"
+		(property "Reference" "C34"
 			(at 151.13 127.508 0)
 			(effects
@@
 			(project "Remora Nucleo F446ZE Hat"
 				(path "/5473abc6-7b93-43cc-a401-f691c4d7d7cf/5cdad347-c6ad-4791-9d53-e4d1ad999196"
-					(reference "C22")
+					(reference "C34")
 					(unit 1)
 				)
@@
 		(on_board yes)
 		(dnp no)
-		(property "Reference" "#PWR0154"
+		(property "Reference" "#PWR0222"
 			(at 171.45 143.51 0)
 			(effects
@@
 			(project "Remora Nucleo F446ZE Hat"
 				(path "/5473abc6-7b93-43cc-a401-f691c4d7d7cf/5cdad347-c6ad-4791-9d53-e4d1ad999196"
-					(reference "#PWR0154")
-					(unit 1)
-				)
+					(reference "#PWR0222")
+					(unit 1)
+				)

Commit message: indiscriminate routing, placement experiments, etc
Other:
- moved on the sheet: C34, C35, C36, C37, F11, J25, Q1, R91, R92, R93, R94, R95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

Commit message: Caught some errors with spacing of jumpers, did some BOM consolidation and included BOM. Updates to Gerbers to reflect new changes.
Parts:
- J25: Digikey Part Number 1818-QT02ADP83V0000G-ND -> 732-691412120002B-ND; Digikey URL https://www.digikey.com.au/en/products/detail/amphenol-anyt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 -> https://www.digikey.com.au/en/products/detail/w%C3%BCrth-el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
- U17: Digikey Part Number (none) -> 160-2255-1-ND
Changed lines of the file:
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@@
+			)
+		)
+		(property "Digikey Part Number" "160-2255-1-ND"
+			(at 85.09 123.19 0)
+			(effects
+				(font
+					(size 1.27 1.27)
+				)
 			)
 		)
@@
 			)
 		)
-		(property "Digikey Part Number" "1818-QT02ADP83V0000G-ND"
+		(property "Digikey Part Number" "732-691412120002B-ND"
 			(at 204.47 134.62 0)
 			(effects
@@
 			)
 		)
-		(property "Digikey URL" "https://www.digikey.com.au/en/products/detail/amphenol-anytek/QT02ADP83V0000G/25618889"
+		(property "Digikey URL" "https://www.digikey.com.au/en/products/detail/w%C3%BCrth-elektronik/691412120002B/11478592"
 			(at 204.47 134.62 0)
 			(effects

Commit message: Some file changes and output new gerbers + BOM and centroid file for PCBWay Order
Parts:
- U17: Digikey URL (none) -> https://www.digikey.com.au/en/products/detail/lite-on-inc/l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
- renumbered R97 to R100, R98 to R101, R91 to R94, R92 to R95, R93 to R96, R94 to R97, R95 to R98, R96 to R99
Changed lines of the file:
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@@
 		(on_board yes)
 		(dnp no)
-		(property "Reference" "R94"
+		(property "Reference" "R97"
 			(at 132.08 128.778 90)
 			(effects
@@
 			(project "Remora Nucleo F446ZE Hat"
 				(path "/5473abc6-7b93-43cc-a401-f691c4d7d7cf/5cdad347-c6ad-4791-9d53-e4d1ad999196"
-					(reference "R94")
+					(reference "R97")
 					(unit 1)
 				)
@@
 		(on_board yes)
 		(dnp no)
-		(property "Reference" "R93"
+		(property "Reference" "R96"
 			(at 109.22 128.778 90)
 			(effects
@@
 			(project "Remora Nucleo F446ZE Hat"
 				(path "/5473abc6-7b93-43cc-a401-f691c4d7d7cf/5cdad347-c6ad-4791-9d53-e4d1ad999196"
-					(reference "R93")
+					(reference "R96")
 					(unit 1)
 				)
@@
 					(size 1.27 1.27)
 				)
+				(hide yes)
+			)
+		)
+		(property "Digikey URL" "https://www.digikey.com.au/en/products/detail/lite-on-inc/ltv-247/4307982"
+			(at 85.09 123.19 0)
+			(effects
+				(font
+					(size 1.27 1.27)
+				)
+				(hide yes)
 			)
 		)
@@
 		(on_board yes)
 		(dnp no)
-		(property "Reference" "R96"
+		(property "Reference" "R99"
 			(at 146.812 83.566 0)
 			(effects
@@
 			(project "Remora Nucleo F446ZE Hat"
 				(path "/5473abc6-7b93-43cc-a401-f691c4d7d7cf/5cdad347-c6ad-4791-9d53-e4d1ad999196"
-					(reference "R96")
+					(reference "R99")
 					(unit 1)
 				)
@@
 		(on_board yes)
 		(dnp no)
-		(property "Reference" "R97"
+		(property "Reference" "R100"
 			(at 166.878 143.51 90)
 			(effects
@@
 			(project "Remora Nucleo F446ZE Hat"
 				(path "/5473abc6-7b93-43cc-a401-f691c4d7d7cf/5cdad347-c6ad-4791-9d53-e4d1ad999196"
-					(reference "R97")
+					(reference "R100")
 					(unit 1)
 				)
@@
 		(on_board yes)
 		(dnp no)
-		(property "Reference" "R98"
+		(property "Reference" "R101"
 			(at 178.816 42.926 0)
 			(effects
@@
 			(project "Remora Nucleo F446ZE Hat"
 				(path "/5473abc6-7b93-43cc-a401-f691c4d7d7cf/5cdad347-c6ad-4791-9d53-e4d1ad999196"
-					(reference "R98")
+					(reference "R101")
 					(unit 1)
 				)
@@
 		(on_board yes)
 		(dnp no)
-		(property "Reference" "R91"
+		(property "Reference" "R94"
 			(at 66.294 115.57 90)
 			(effects
@@
 			(project "Remora Nucleo F446ZE Hat"
 				(path "/5473abc6-7b93-43cc-a401-f691c4d7d7cf/5cdad347-c6ad-4791-9d53-e4d1ad999196"
-					(reference "R91")
+					(reference "R94")
 					(unit 1)
 				)
@@
 		(on_board yes)
 		(dnp no)
-		(property "Reference" "R95"
+		(property "Reference" "R98"
 			(at 153.162 58.166 90)
 			(effects
@@
 			(project "Remora Nucleo F446ZE Hat"
 				(path "/5473abc6-7b93-43cc-a401-f691c4d7d7cf/5cdad347-c6ad-4791-9d53-e4d1ad999196"
-					(reference "R95")
+					(reference "R98")
 					(unit 1)
 				)
@@
 		(on_board yes)
 		(dnp no)
-		(property "Reference" "R92"
+		(property "Reference" "R95"
 			(at 103.378 139.7 90)
 			(effects
@@
 			(project "Remora Nucleo F446ZE Hat"
 				(path "/5473abc6-7b93-43cc-a401-f691c4d7d7cf/5cdad347-c6ad-4791-9d53-e4d1ad999196"
-					(reference "R92")
-					(unit 1)
-				)
+					(reference "R95")
+					(unit 1)
+				)
